File: Hardware/APMC.kicad_pcb (KiCad board)
At the start: 2 copper layers, 85 x 52.5 mm, 151 parts, among them J1 Pin header Male 2x7 P:1.27, J10 +3.3V, J11 +3.3V, J13 +3.3V, J14 Conn_01x04, J2 USB-C, J5 Terminal 1x5 P:3.5mm, J6 Terminal 1x5 P:3.5mm, J7 Terminal 1x5 P:3.5mm, J8 Conn_01x04, J9 Conn_01x04, M1 Logo_Open_Hardware_Small, Q1 DMP6023LE, Q10 BSS123, Q2 DMP6023LE, Q3 DMP6023LE, Q4 BSS123, Q5 DMP6023LE, Q6 DMP6023LE, Q7 BSS123, Q8 DMP3056L, Q9 BSS123, U1 LMR516xx, U10 TXU0202, U12 LM74703/LM74704, U13 TPS62162DSG, U2 LCFE201202A, U3 TXU0202, U4 M95P32, U5 STM32U575CITx, U6 XTR200, U7 TPS7A2031PDBVR, U8 XTR200, U9 ADS1x2S14, X1 SiT8008Bx-7x, Y1 32.768kHz

Commit message: BOM revised
Parts:
- J10, J11, J13: value +3.3V -> Conn_01x03
- J12: value ~ -> Conn_02x08
- J2: value USB-C -> USB-C receptacle
- R28: value 300k -> 681k
- R33: value 300k -> 1.5M
- R35: value 300k -> X
Connections:
- net Net-(U1-SW) renamed /SW
- net VDDA renamed /VDDA
Routing:
- net GND: track 92.6 -> 91.8 mm, vias 327 -> 332

Commit message: schematic fix
Connections:
- Q1 pad 2: /VIN -> /VCC
- Q1 pad 3: /VCC -> /VIN

Commit message: R19 fix
Parts:
- C49, C50: value 22uF/10V -> 22uF/6.3V
- R12, R13: value 4.7k -> 4.3k
- R19: value 5.1k -> 4.3k
Changed lines of the file:
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@@
 			)
 		)
-		(property "Angle55" ""
-			(at 0 0 90)
-			(unlocked yes)
-			(layer "F.Fab")
-			(hide yes)
-			(effects
-				(font
-					(size 1 1)
-					(thickness 0.15)
-				)
-			)
-		)
-		(property "Vertical" ""
-			(at 0 0 90)
-			(unlocked yes)
-			(layer "F.Fab")
-			(hide yes)
-			(effects
-				(font
-					(size 1 1)
-					(thickness 0.15)
-				)
-			)
-		)
-		(property "AliExpress" ""
-			(at 0 0 90)
-			(unlocked yes)
-			(layer "F.Fab")
-			(hide yes)
-			(effects
-				(font
-					(size 1 1)
-					(thickness 0.15)
-				)
-			)
-		)
-		(property "Source" ""
-			(at 0 0 90)
-			(unlocked yes)
-			(layer "F.Fab")
-			(hide yes)
-			(effects
-				(font
-					(size 1 1)
-					(thickness 0.15)
-				)
-			)
-		)
-		(property "ST reccomended" ""
+		(property "Note" "consider using LM66100 in SC-70-6 pkg instead"
 			(at 0 0 90)
 			(unlocked yes)
@@
 			)
 		)
-		(property "Notes" "Vds 80V min, Vgs(th) ~1.5V, Rds(on) ≤ 10Ω"
-			(at 0 0 0)
-			(unlocked yes)
-			(layer "F.Fab")
-			(hide yes)
-			(effects
-				(font
-					(size 1 1)
-					(thickness 0.15)
-				)
-			)
-		)
-		(property "Angle55" ""
-			(at 0 0 0)
-			(unlocked yes)
-			(layer "F.Fab")
-			(hide yes)
-			(effects
-				(font
-					(size 1 1)
-					(thickness 0.15)
-				)
-			)
-		)
-		(property "Vertical" ""
-			(at 0 0 0)
-			(unlocked yes)
-			(layer "F.Fab")
-			(hide yes)
-			(effects
-				(font
-					(size 1 1)
-					(thickness 0.15)
-				)
-			)
-		)
-		(property "AliExpress" ""
-			(at 0 0 0)
-			(unlocked yes)
-			(layer "F.Fab")
-			(hide yes)
-			(effects
-				(font
-					(size 1 1)
-					(thickness 0.15)
-				)
-			)
-		)
-		(property "Source" ""
-			(at 0 0 0)
-			(unlocked yes)
-			(layer "F.Fab")
-			(hide yes)
-			(effects
-				(font
-					(size 1 1)
-					(thickness 0.15)
-				)
-			)
-		)
-		(property "ST reccomended" ""
+		(property "Notes" "Vds(max) ≥ 30V, Vgs(th) ~1.5V, Vgs(max) ≥ ±20V, Rds(on) ≤ 10Ω"
 			(at 0 0 0)
 			(unlocked yes)
@@
 			)
 		)
-		(property "Notes" "Vds 80V min, Vgs(th) ~1.5V, Rds(on) ≤ 10Ω"
-			(at 0 0 0)
-			(unlocked yes)
-			(layer "F.Fab")
-			(hide yes)
-			(effects
-				(font
-					(size 1 1)
-					(thickness 0.15)
-				)
-			)
-		)
-		(property "Angle55" ""
-			(at 0 0 0)
-			(unlocked yes)
-			(layer "F.Fab")
-			(hide yes)
-			(effects
-				(font
-					(size 1 1)
-					(thickness 0.15)
-				)
-			)
-		)
-		(property "Vertical" ""
-			(at 0 0 0)
-			(unlocked yes)
-			(layer "F.Fab")
-			(hide yes)
-			(effects
-				(font
-					(size 1 1)
-					(thickness 0.15)
-				)
-			)
-		)
-		(property "AliExpress" ""
-			(at 0 0 0)
-			(unlocked yes)
-			(layer "F.Fab")
-			(hide yes)
-			(effects
-				(font
-					(size 1 1)
-					(thickness 0.15)
-				)
-			)
-		)
-		(property "Source" ""
-			(at 0 0 0)
-			(unlocked yes)
-			(layer "F.Fab")
-			(hide yes)
-			(effects
-				(font
-					(size 1 1)
-					(thickness 0.15)
-				)
-			)
-		)
-		(property "ST reccomended" ""
+		(property "Notes" "Vds(max) ≥ 30V, Vgs(th) ~1.5V, Vgs(max) ≥ ±20V, Rds(on) ≤ 10Ω"
 			(at 0 0 0)
 			(unlocked yes)
@@
 			)
 		)
-		(property "Value" "4.7k"
+		(property "Value" "4.3k"
 			(at 0 1.43 90)
 			(layer "F.Fab")
@@
 			)
 		)
-		(property "Mfg" "Susumu: RG1608P-472-D-T5"
+		(property "Mfg" "Susumu: RR0816P-432-D"
 			(at 0 0 270)
 			(unlocked yes)
@@
 			)
 		)
-		(property "Mouser" "754-RG1608P-472DT5"
+		(property "Mouser" "754-RR0816P-432D"
 			(at 0 0 270)
 			(unlocked yes)
@@
 			)
 		)
-		(property "Value" "4.7k"
+		(property "Value" "4.3k"
 			(at 0 1.43 90)
 			(layer "F.Fab")
@@
 			)
 		)
-		(property "Mfg" "Susumu: RG1608P-472-D-T5"
+		(property "Mfg" "Susumu: RR0816P-432-D"
 			(at 0 0 270)
 			(unlocked yes)
@@
 			)
 		)
-		(property "Mouser" "754-RG1608P-472DT5"
+		(property "Mouser" "754-RR0816P-432D"
 			(at 0 0 270)
 			(unlocked yes)
@@
 			)
 		)
-		(property "Value" "5.1k"
+		(property "Value" "4.3k"
 			(at 0 1.43 0)
 			(layer "F.Fab")
@@
 			)
 		)
-		(property "Mfg" "Susumu: RR0816P-512-D"
+		(property "Mfg" "Susumu: RR0816P-432-D"
 			(at 0 0 0)
 			(unlocked yes)
@@
 			)
 		)
-		(property "Mouser" "754-RR0816P-512D"
+		(property "Mouser" "754-RR0816P-432D"
 			(at 0 0 0)
 			(unlocked yes)
@@
 			)
 		)
-		(property "Value" "22uF/10V"
+		(property "Value" "22uF/6.3V"
 			(at 0 1.85 90)
 			(layer "F.Fab")
@@
 			)
 		)
-		(property "Value" "22uF/10V"
+		(property "Value" "22uF/6.3V"
 			(at 0 1.85 0)
 			(layer "F.Fab")

Commit message: label fix
Changed lines of the file:
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@@
 			)
 		)
-		(property "Label" "VDD"
+		(property "Label" "3.3V"
 			(at -2.125 0 0)
 			(unlocked yes)
@@
 			)
 		)
-		(property "Label" "3V 5V"
+		(property "Label" "3.3V 5V"
 			(at 0 1.875 0)
 			(unlocked yes)
@@
 			)
 		)
-		(property "Label" "3V 5V"
+		(property "Label" "3.3V 5V"
 			(at 0 1.875 0)
 			(unlocked yes)
@@
 			)
 		)
-		(property "Label" "3V 5V"
+		(property "Label" "3.3V 5V"
 			(at 0 1.875 0)
 			(unlocked yes)

Commit message: post-prod updates
Parts:
- removed C31, C36, C38, C43: 10nF, Custom:C_0603_1608Metric_Pad0.98x0.95mm_HandSolder
- removed C57: 100nF, Custom:C_0603_1608Metric_Pad0.98x0.95mm_HandSolder
- removed Q10, Q9: BSS123, Package_TO_SOT_SMD:SOT-323_SC-70
- removed R16, R41: 3.3k, Resistor_SMD:R_0603_1608Metric_Pad0.98x0.95mm_HandSolder
- added C33: 10nF, Custom:RC_Array_Isolated_4_0805, F.Cu at (45.8, 60.5)
- added C58: 100nF, Capacitor_SMD:C_0603_1608Metric_Pad1.08x0.95mm_HandSolder, F.Cu at (86.0, 53.1)
- added R24: 3.3k, Resistor_SMD:R_0603_1608Metric_Pad0.98x0.95mm_HandSolder, F.Cu at (94.8, 56.4)
- added R25: 3.3k, Resistor_SMD:R_0603_1608Metric_Pad0.98x0.95mm_HandSolder, F.Cu at (96.1, 56.4)
- added R29: 100k, Resistor_SMD:R_0603_1608Metric_Pad0.98x0.95mm_HandSolder, F.Cu at (89.8, 55.6)
- added U11: PCA9306, Custom:VSSOP-8_2.3x2mm_P0.5mm, F.Cu at (86.6, 55.1)
- H1, H2, H3, H4: value MountingHole -> M2.5x7
- R21, R28, R33, R35: footprint Resistor_SMD:R_0603_1608Metric_Pad0.98x0.95mm_HandSolder -> Resistor_SMD:R_0805_2012Metric
- U4: footprint Custom:DFN-8-1EP_4x4mm_P0.8mm_EP2.2x3.2mm -> Package_SO:SO-8_3.9x4.9mm_P1.27mm
- U9: footprint Package_DFN_QFN:WQFN-16-1EP_3x3mm_P0.5mm_EP1.68x1.68mm_ThermalVias -> Custom:WQFN-16-1EP_3x3mm_P0.5mm_EP1.68x1.68mm_ThermalVias
- moved R46 7.25 mm to (49.5, 14.1)
- moved C8 4.81 mm to (58.4, 45.5)
- moved R6 2.77 mm to (65.4, 43.6)
- moved R20 2.10 mm to (38.6, 52.6)
- moved R21 2.10 mm to (42.0, 52.6)
- moved U4 1.68 mm to (61.9, 45.5)
- moved R27 1.40 mm to (38.6, 54.6)
- moved R28 1.40 mm to (42.0, 54.6)
- moved C41 0.91 mm to (93.4, 56.4)
- moved R32 0.80 mm to (38.6, 56.6)
- moved R33 0.80 mm to (42.0, 56.6)
- moved R34 0.67 mm to (38.6, 58.6)
- moved R35 0.67 mm to (42.0, 58.6)
- moved C29 0.64 mm to (49.0, 55.9)
- moved Q1 0.62 mm to (45.4, 17.5), turned to 0 degrees
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Routing:
- net /VCC: track 87.4 -> 79.2 mm
- net /VIN: track 22.2 -> 30.1 mm, vias 0 -> 2
- net /ADC0: track 70.0 -> 63.0 mm
- net Net-(Q1-G): track 5.02 -> 10.4 mm
- net GND: track 91.8 -> 86.6 mm, vias 332 -> 330
- net /VDD: track 281.9 -> 277.1 mm
- net /VDDA: track 54.1 -> 49.9 mm
- net /SDA: track 9.58 -> 12.7 mm
- net /5V: track 106.9 -> 104.3 mm
- net /ADC3: track 9.74 -> 12.1 mm
- net /VIN1: track 8.17 -> 5.84 mm
- net Net-(U11-EN): track 0.00 -> 1.91 mm
- net Net-(D12-A): track 7.95 -> 6.11 mm
- net Net-(C3-Pad2): track 25.7 -> 23.9 mm
- net Net-(D5-A): track 13.5 -> 11.8 mm
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Other:
- board text added: "All-purpose Micro Controller (APMC) rev. 2.0.1 2026-07-21"
- board text removed: "All-purpose Micro Controller (APMC) rev. 2.0 2026-07-15"

Commit message: post-prod fixes
Parts:
- C51, C53, C55, C56, C58: footprint Capacitor_SMD:C_0603_1608Metric_Pad1.08x0.95mm_HandSolder -> Custom:C_0603_1608Metric_Pad0.98x0.95mm_HandSolder
- moved M1 8.50 mm to (56.5, 61.8)
- moved C9 7.87 mm to (52.0, 28.9), turned to 90 degrees
- moved R24 3.35 mm to (97.8, 54.9), turned to 90 degrees
- moved Q4 3.28 mm to (57.9, 32.1), turned to 90 degrees
- moved R10 2.46 mm to (55.0, 33.0), turned to 180 degrees
- moved C51 2.25 mm to (81.0, 55.9), turned to 180 degrees
- moved C55 2.25 mm to (64.0, 55.9), turned to 180 degrees
- moved C41 2.03 mm to (94.8, 54.9), turned to 90 degrees
- moved C58 1.86 mm to (84.6, 51.9)
- moved R29 1.86 mm to (88.4, 54.4)
- moved U11 1.86 mm to (85.2, 53.9)
- moved R25 1.51 mm to (96.2, 54.9), turned to 90 degrees
- moved D5 1.25 mm to (54.0, 28.9)
- moved J14 1.25 mm to (61.0, 57.5)
- moved J8 1.25 mm to (95.0, 57.5)
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Routing:
- net /VCC: track 79.2 -> 67.6 mm
- net /VDD1: track 19.5 -> 25.4 mm, vias 1 -> 2
- net GND: track 86.6 -> 90.3 mm, vias 330 -> 334
- net /VDD: track 277.1 -> 280.6 mm
- net /PWM1: track 35.8 -> 32.7 mm
- net Net-(D5-A): track 11.8 -> 13.7 mm
- net /I2C_SDA: track 31.9 -> 30.1 mm
- net /I2C_SCL: track 30.5 -> 28.7 mm
- net /PWM2: track 33.5 -> 32.0 mm
- net /UART_TX: track 24.5 -> 23.3 mm
- net /UART_RX: track 24.8 -> 23.5 mm
- net /FDCAN_TX: track 24.9 -> 23.6 mm
- net /FDCAN_RX: track 23.6 -> 22.3 mm
- net /VDD2: track 15.4 -> 16.6 mm
- net /SDA: track 12.7 -> 11.6 mm
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
Commit message: post-prod fixes
Parts:
- FB1, FB2: footprint Fuse:Fuse_1210_3225Metric_Pad1.42x2.65mm_HandSolder -> Fuse:Fuse_1206_3216Metric_Pad1.42x1.75mm_HandSolder
- moved C44 1.91 mm to (99.0, 21.9)
- moved Q4 0.53 mm to (57.5, 32.5)
- moved R10 0.53 mm to (54.6, 33.4)
- moved R8 0.53 mm to (54.6, 31.9)
- moved FB1 0.52 mm to (54.5, 24.8)
- moved FB2 0.50 mm to (70.8, 25.6)
- moved R15 0.38 mm to (52.2, 32.5)
- moved D5 0.25 mm to (54.0, 29.1)
- moved J4 0.25 mm to (75.5, 25.2)
- moved R7 0.25 mm to (55.6, 29.1)
- moved C49 0.19 mm to (63.9, 25.6)
- moved R3 0.18 mm to (87.1, 18.4)
- moved C9 0.12 mm to (52.1, 28.9)
- moved Q7 0.12 mm to (54.6, 35.6)
Routing:
- net /STLINK_TX: track 24.4 -> 22.2 mm
- net /VDD: track 280.6 -> 279.2 mm
- net /VDD1: track 25.4 -> 26.6 mm
- net Net-(D5-A): track 13.7 -> 13.0 mm
- net GND: track 90.3 -> 89.8 mm
