File: Hardware/APMC.kicad_pcb (KiCad board)
At the start: 2 copper layers, 85 x 52.5 mm, 148 parts, among them J1 Pin header Male 2x7 P:1.27, J10 Conn_01x03, J11 Conn_01x03, J12 Conn_02x08, J13 Conn_01x03, J14 Conn_01x04, J2 USB-C receptacle, J5 Terminal 1x5 P:3.5mm, J6 Terminal 1x5 P:3.5mm, J7 Terminal 1x5 P:3.5mm, J8 Conn_01x04, J9 Conn_01x04, M1 Logo_Open_Hardware_Small, Q1 DMP6023LE, Q2 DMP6023LE, Q3 DMP6023LE, Q4 BSS123, Q5 DMP6023LE, Q6 DMP6023LE, Q7 BSS123, Q8 DMP3056L, U1 LMR516xx, U10 TXU0202, U11 PCA9306, U12 LM74703/LM74704, U13 TPS62162DSG, U2 LCFE201202A, U3 TXU0202, U4 M95P32, U5 STM32U575CITx, U6 XTR200, U7 TPS7A2031PDBVR, U8 XTR200, U9 ADS1x2S14, X1 SiT8008Bx-7x, Y1 32.768kHz

Commit message: post-prod fixes
Parts:
- C28: value 1uF/4V -> 4.7uF/4V; footprint Capacitor_SMD:C_0603_1608Metric_Pad1.08x0.95mm_HandSolder -> Custom:C_0603_1608Metric_Pad0.98x0.95mm_HandSolder
- L1: value 15uH -> 33uH
- U1: value LMR516xx -> LMR51610
- turned C28 to 90 degrees
Connections:
- C28 pad 1: /VDDA -> GND
- C28 pad 2: GND -> /VDDA

Commit message: initial firmware
Parts:
- J1: footprint Custom:PinHeader_2x07_P1.27mm_Horizontal -> Custom:PinHeader_2x07_P1.27mm_Horizontal-UP
- moved R3 7.87 mm to (94.6, 20.8), turned to 0 degrees
Routing:
- net /STLINK_TX: track 22.2 -> 33.2 mm
- net /NRST: track 62.8 -> 59.5 mm
- net /VDD: track 279.2 -> 282.4 mm
- net /SWDIO: track 28.5 -> 26.9 mm
- net Net-(J1-Pin_11): track 2.91 -> 1.76 mm
- net /SWCLK: track 29.3 -> 30.4 mm
- net GND: vias 334 -> 333
Other:
- outline, holes or cut-outs redrawn

Commit message: initial firmware version working
Parts:
- moved D7 0.88 mm to (83.9, 23.5)
- moved J2 0.88 mm to (79.5, 19.9)
- moved J4 0.88 mm to (75.5, 26.1)
- moved Q8 0.88 mm to (74.6, 23.2)
- moved R1 0.88 mm to (80.9, 23.5)
- moved R2 0.88 mm to (77.1, 23.5)
- moved R9 0.88 mm to (82.4, 23.5)
- moved U2 0.88 mm to (79.0, 23.5)
Routing:
- net /VDD: track 282.4 -> 281.6 mm, vias 7 -> 8
- net /STATUS_LED: track 15.1 -> 14.4 mm
- net GND: vias 333 -> 332

Commit message: DBCC fix
Routing:
- net /C: track 24.5 -> 23.9 mm
- net GND: vias 332 -> 330
- net /VDD: vias 8 -> 7

Commit message: LVGL timer fix
Parts:
- moved D7 5.54 mm to (86.2, 18.5), turned to -90 degrees
- moved R9 2.91 mm to (85.0, 22.2), turned to 180 degrees
Routing:
- net /STATUS_LED: track 14.4 -> 22.2 mm
- net /VDD: track 281.6 -> 284.5 mm
- net Net-(D7-A): track 1.50 -> 2.98 mm
- net GND: vias 330 -> 328
