File: Hardware/APMC.kicad_sch (KiCad schematic)
At the start: 157 parts, among them J1 Pin header Male 2x7 P:1.27, J10 Conn_01x03, J11 Conn_01x03, J12 Conn_02x08, J13 Conn_01x03, J14 Conn_01x04, J2 USB-C receptacle, J5 Terminal 1x5 P:3.5mm, J6 Terminal 1x5 P:3.5mm, J7 Terminal 1x5 P:3.5mm, J8 Conn_01x04, J9 Conn_01x04, M1 Logo_Open_Hardware_Small, Q1 DMP6023LE, Q2 DMP6023LE, Q3 DMP6023LE, Q4 BSS123, Q5 DMP6023LE, Q6 DMP6023LE, Q7 BSS123, Q8 DMP3056L, U1 LMR516xx, U10 TXU0202, U11 PCA9306, U12 LM74703/LM74704, U13 TPS62162DSG, U2 LCFE201202A, U3 TXU0202, U4 M95P32, U5 STM32U575CITx, U6 XTR200, U7 TPS7A2031PDBVR, U8 XTR200, U9 ADS1x2S14, X1 SiT8008Bx-7x, Y1 32.768kHz

Commit message: BOM fix
Parts:
- R21: Mfg Panasonic: ERA-3AEB304V -> Susumu: RG2012P-304-B-T5; Mouser 667-ERA-3AEB304V -> 754-RG2012P-304-BT5
- R28: Mfg Yageo: RT0603BRD07681KL -> Panasonic: ERA-6AEB6813V; Mouser 603-RT0603BRD07681KL -> 667-ERA-6AEB6813V
- R33: Mfg Vishay: MCT0603MD1504BP500 -> Susumu: RG2012P-155-B-T5; Mouser 594-MCT0603MD1504BP5 -> 754-RG2012P-155B-T5
Changed lines of the file:
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@@
 			)
 		)
-		(property "Mfg" "Yageo: RT0603BRD07681KL"
+		(property "Mfg" "Panasonic: ERA-6AEB6813V"
 			(at 49.53 143.51 0)
 			(hide yes)
@@
 			)
 		)
-		(property "Mouser" "603-RT0603BRD07681KL"
+		(property "Mouser" "667-ERA-6AEB6813V"
 			(at 49.53 143.51 0)
 			(hide yes)
@@
 			)
 		)
-		(property "Mfg" "Vishay: MCT0603MD1504BP500"
+		(property "Mfg" "Susumu: RG2012P-155-B-T5"
 			(at 49.53 161.29 0)
 			(hide yes)
@@
 			)
 		)
-		(property "Mouser" "594-MCT0603MD1504BP5"
+		(property "Mouser" "754-RG2012P-155B-T5"
 			(at 49.53 161.29 0)
 			(hide yes)
@@
 			)
 		)
-		(property "Angle55" ""
-			(at 39.37 143.51 90)
-			(hide yes)
-			(show_name no)
-			(do_not_autoplace no)
-			(effects
-				(font
-					(size 1.27 1.27)
-				)
-			)
-		)
-		(property "Vertical" ""
-			(at 39.37 143.51 90)
-			(hide yes)
-			(show_name no)
-			(do_not_autoplace no)
-			(effects
-				(font
-					(size 1.27 1.27)
-				)
-			)
-		)
-		(property "AliExpress" ""
-			(at 39.37 143.51 90)
-			(hide yes)
-			(show_name no)
-			(do_not_autoplace no)
-			(effects
-				(font
-					(size 1.27 1.27)
-				)
-			)
-		)
-		(property "Source" ""
-			(at 39.37 143.51 90)
-			(hide yes)
-			(show_name no)
-			(do_not_autoplace no)
-			(effects
-				(font
-					(size 1.27 1.27)
-				)
-			)
-		)
-		(property "ST reccomended" ""
-			(at 39.37 143.51 90)
-			(hide yes)
-			(show_name no)
-			(do_not_autoplace no)
-			(effects
-				(font
-					(size 1.27 1.27)
-				)
-			)
-		)
 		(pin "1"
 		)
@@
 			)
 		)
-		(property "Angle55" ""
-			(at 39.37 161.29 90)
-			(hide yes)
-			(show_name no)
-			(do_not_autoplace no)
-			(effects
-				(font
-					(size 1.27 1.27)
-				)
-			)
-		)
-		(property "Vertical" ""
-			(at 39.37 161.29 90)
-			(hide yes)
-			(show_name no)
-			(do_not_autoplace no)
-			(effects
-				(font
-					(size 1.27 1.27)
-				)
-			)
-		)
-		(property "AliExpress" ""
-			(at 39.37 161.29 90)
-			(hide yes)
-			(show_name no)
-			(do_not_autoplace no)
-			(effects
-				(font
-					(size 1.27 1.27)
-				)
-			)
-		)
-		(property "Source" ""
-			(at 39.37 161.29 90)
-			(hide yes)
-			(show_name no)
-			(do_not_autoplace no)
-			(effects
-				(font
-					(size 1.27 1.27)
-				)
-			)
-		)
-		(property "ST reccomended" ""
-			(at 39.37 161.29 90)
-			(hide yes)
-			(show_name no)
-			(do_not_autoplace no)
-			(effects
-				(font
-					(size 1.27 1.27)
-				)
-			)
-		)
 		(pin "1"
 		)
@@
 			)
 		)
-		(property "Angle55" ""
-			(at 39.37 177.8 90)
-			(hide yes)
-			(show_name no)
-			(do_not_autoplace no)
-			(effects
-				(font
-					(size 1.27 1.27)
-				)
-			)
-		)
-		(property "Vertical" ""
-			(at 39.37 177.8 90)
-			(hide yes)
-			(show_name no)
-			(do_not_autoplace no)
-			(effects
-				(font
-					(size 1.27 1.27)
-				)
-			)
-		)
-		(property "AliExpress" ""
-			(at 39.37 177.8 90)
-			(hide yes)
-			(show_name no)
-			(do_not_autoplace no)
-			(effects
-				(font
-					(size 1.27 1.27)
-				)
-			)
-		)
-		(property "Source" ""
-			(at 39.37 177.8 90)
-			(hide yes)
-			(show_name no)
-			(do_not_autoplace no)
-			(effects
-				(font
-					(size 1.27 1.27)
-				)
-			)
-		)
-		(property "ST reccomended" ""
-			(at 39.37 177.8 90)
-			(hide yes)
-			(show_name no)
-			(do_not_autoplace no)
-			(effects
-				(font
-					(size 1.27 1.27)
-				)
-			)
-		)
 		(pin "1"
 		)
@@
 			)
 		)
-		(property "Mfg" "Panasonic: ERA-3AEB304V"
+		(property "Mfg" "Susumu: RG2012P-304-B-T5"
 			(at 49.53 127 0)
 			(hide yes)
@@
 			)
 		)
-		(property "Mouser" "667-ERA-3AEB304V"
+		(property "Mouser" "754-RG2012P-304-BT5"
 			(at 49.53 127 0)
 			(hide yes)
@@
 			(hide yes)
 			(show_name no)
-			(do_not_autoplace no)
-			(effects
-				(font
-					(size 1.27 1.27)
-				)
-			)
-		)
-		(property "ST reccomended" ""
-			(at 49.53 177.8 90)
-			(hide yes)
-			(show_name no)

Commit message: post-prod fixes
Parts:
- C19: Remarks ESR < 20 mΩ at 3 MHz -> ESR < 20 mΩ @ 3 MHz
- C51, C53, C55, C56, C58: footprint Capacitor_SMD:C_0603_1608Metric_Pad1.08x0.95mm_HandSolder -> Custom:C_0603_1608Metric_Pad0.98x0.95mm_HandSolder
- L2: Ferrite CDPH4D19FNP-3R3MC, LPS6225-332MRC, LPS5030-332MRC, MSS5121-332MLC, MSS5131-332MLC, SD25-3R3-R, 74408053003, SD53-3R3-R -> CDPH4D19FNP-3R3MC, LPS6225-332MRC, LPS5030-332MRC, MSS5121-332MLC, MSS5131-332MLC, SD25-3R3-R, 74408053003, SD53-3R3-R, ASPI-0628-3R3M-T1, PG0087.332NLT; Mfg Sumida: CDPH4D19FNP-3R3MC -> Bourns: SRR5828A-3R3Y; Mouser 851-CDPH4D19FNP3R3MC -> 6521-SRR5828A-3R3Y

Commit message: post-prod fixes
Parts:
- FB1, FB2: footprint Fuse:Fuse_1210_3225Metric_Pad1.42x2.65mm_HandSolder -> Fuse:Fuse_1206_3216Metric_Pad1.42x1.75mm_HandSolder
- L1: value 15uH -> 33uH; 10x10 DD1274AS-H-150M=P3 (5mm), 7447714150 (5mm) -> DD1274AS-H-330M=P3, MSS1048-333MLC, CDRH104NP-330MC, 744771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; B2 DEM8045Z-150M=P3 -> (none); Ferrite 8x8 IFSC3232DBER150M01, SRN8040HA-150M, BWVS00808040150M00, SRN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 -> CDRH8D28NP-330NC, CDRH8D28NP-330NC, CDRH8D43HPNP-330NC, SCR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; Mfg Murata: DEM8045Z-150M=P3 -> Murata: 1248AS-H-330M=P3; Mouser 81-DEM8045Z-150M=P3 -> 81-1248AS-H-330MP3; Murata 8x8 1248AS-H-150M=P3, DEM8045Z-150M=P3 -> DEM8045Z-330M=P3, 1248AS-H-330M=P3
- R45: Remarks 0.5% -> 0.5%, use 21k for 6V lower range (Susumu: RG1608P-2102-D-T5)
- U1: value LMR516xx -> LMR51610; symbol LMR516xx:LMR516xx -> LMR51610:LMR51610; Alt (none) -> LMR51610XFDBVR, LMR51606XDBVR, LMR51606XFDBVR, LMR51606XQDB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; Alt2 (none) -> pin-compatible, Vin 36V max: LMR50410 (700kHz), TPS560430 (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; Mfg TI: LMR51625XDDCR -> TI: LMR51610XDBVR; Mouser 595-LMR51625XDDCR -> 595-LMR51610XDBVR; Remarks SPREAD SPECTRUM & PFM -> PFM 400kHz version, do not use LMR51625 or LMR51635 (differ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
- U13: Alt2 (none) -> TPS560430X3F (SOT-23 3.3V)
Other:
- note removed: "LMR51610 (33uH) LMR51625 (15uH) LMR51635 (8.2uH)"
